File: Électrique/Module Central/Module Central.kicad_pcb (KiCad board)
At the start: 2 copper layers, 48.2 x 45.8 mm, 48 parts, among them J101 2.1mm X 5.5mm Barrel Connector, J102 Prog, J103 Conn_Coaxial, J201 USB_B_Mini, J301 Borne 0, J302 Borne 1, J303 Borne 2, J304 Borne 3, U101 LM2937xMP, U102 ATmega328P-AU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

Commit message: MAJ liste pieces
Other:
- board text added: "1W"
